Commit message: chapter M(진행중): URDF에 inertial·collision 추가 + Gazebo 설치

File: ros2_ws/src/fake_robot/urdf/fake_robot.urdf.xacro (robot description, xacro)
@@ -4,4 +4,8 @@
     <xacro:property name="track" value="0.4" />
     <xacro:property name="caster_radius" value="0.03" />
+    <xacro:property name="body_x" value="0.4" />
+    <xacro:property name="body_y" value="0.3" />
+    <xacro:property name="body_z" value="0.1" />
+    <xacro:property name="body_mass" value="5.0" />
     <material name="blue">
         <color rgba="0.2 0.4 0.8 1.0" />
@@ -10,4 +14,36 @@
         <color rgba="0.1 0.1 0.1 1.0" />
     </material>
+    <xacro:macro name="box_inertia" params="m w d h">
+        <inertial>
+            <origin xyz="0 0 0" />
+            <mass value="${m}" />
+            <inertia ixx="${m*( d*d + h*h )/12}"
+                iyy="${m*( w*w + h*h )/12}"
+                izz="${m*( w*w + d*d )/12}"
+                ixy="0" ixz="0" iyz="0" />
+        </inertial>
+    </xacro:macro>
+    <xacro:macro name="cylinder_inertia" params="m r l rpy">
+        <inertial>
+            <origin rpy="${rpy}" xyz="0 0 0" />
+            <mass value="${m}" />
+            <inertia ixx="${m * (3 * r * r + l * l) / 12}"
+                iyy="${m * (3 * r * r + l * l) / 12}"
+                izz="${m*r*r/2}"
+                ixy="0" ixz="0" iyz="0" />
+        </inertial>
+    </xacro:macro>
+    <xacro:macro name="sphere_inertia" params="m r">
+        <inertial>
+            <origin xyz="0 0 0" />
+            <mass value="${m}" />
+            <inertia ixx="${2 * m * r * r / 5}"
+                iyy="${2 * m * r * r / 5}"
+                izz="${2 * m * r * r / 5}"
+                ixy="0"
+                ixz="0"
+                iyz="0" />
+        </inertial>
+    </xacro:macro>
     <xacro:macro name="wheel" params="prefix reflect">
         <link name="${prefix}_wheel">
@@ -19,4 +55,11 @@
                 <material name="black" />
             </visual>
+            <collision>
+                <geometry>
+                    <cylinder radius="${wheel_radius}" length="${wheel_width}" />
+                </geometry>
+                <origin rpy="1.5708 0 0" xyz="0 0 0" />
+            </collision>
+            <xacro:cylinder_inertia m="0.5" r="${wheel_radius}" l="${wheel_width}" rpy="1.5708 0 0" />
         </link>
         <joint name="${prefix}_wheel_joint" type="continuous">
@@ -30,8 +73,14 @@
         <visual>
             <geometry>
-                <box size="0.4 0.3 0.1" />
+                <box size="${body_x} ${body_y} ${body_z}" />
             </geometry>
             <material name="blue" />
         </visual>
+        <collision>
+            <geometry>
+                <box size="${body_x} ${body_y} ${body_z}" />
+            </geometry>
+        </collision>
+        <xacro:box_inertia m="${body_mass}" w="${body_x}" d="${body_y}" h="${body_z}" />
     </link>
     <link name="laser">
@@ -42,4 +91,10 @@
             <material name="black" />
         </visual>
+        <collision>
+            <geometry>
+                <cylinder radius="0.03" length="0.04" />
+            </geometry>
+        </collision>
+        <xacro:cylinder_inertia m="0.2" r="0.03" l="0.04" rpy="0 0 0" />
     </link>
     <joint name="laser_joint" type="fixed">
@@ -51,13 +106,19 @@
         <visual>
             <geometry>
-                <sphere radius="${caster_radius}"/>
+                <sphere radius="${caster_radius}" />
             </geometry>
             <material name="black" />
         </visual>
+        <collision>
+            <geometry>
+                <sphere radius="${caster_radius}" />
+            </geometry>
+        </collision>
+        <xacro:sphere_inertia m="0.1" r="${caster_radius}" />
     </link>
     <joint name="caster_joint" type="fixed">
-        <parent link="base_link"/>
-        <child link="caster"/>
-        <origin xyz="-0.15 0 ${-wheel_radius + caster_radius}" rpy ="0 0 0"/>
+        <parent link="base_link" />
+        <child link="caster" />
+        <origin xyz="-0.15 0 ${-wheel_radius + caster_radius}" rpy="0 0 0" />
     </joint>
     <xacro:wheel prefix="left" reflect="1" />

Commit message: chapter M 완료: Gazebo 시뮬 — 물리 엔진 위의 로봇, 레스토랑 월드, 키보드 텔레옵
- URDF: <inertial>/<collision> 채우고 관성 매크로 3종(box/cylinder/sphere)
- Gazebo 플러그인: DiffDrive, JointStatePublisher, gpu_lidar
  - 프레임 접두사 문제를 <frame_id>/<child_frame_id>/<gz_frame_id>로 해결
- 캐스터를 앞뒤 2개로: 무게중심(+0.004)이 지지 구간 밖이라 로봇이 8.8도 앞으로
  넘어져 있었다. 2D 오도메트리는 pitch를 발행하지 않아 TF도 화면도 멀쩡했고,
  손으로 계산한 라이다 기대 거리(3.75m)와 실측(0.92m)의 차이로 발견
- worlds/restaurant.sdf: 시스템 플러그인 5종, 벽 4개(색상 구분), 테이블 4개,
  헤드리스 렌더링용 관전 카메라(지도 시점)
- teleop_node: termios 원시 모드로 엔터 없이 키 입력, 20Hz로 /cmd_vel 발행
  RawTerminal RAII 클래스로 종료 경로와 무관하게 터미널 복원 보장
- CMakeLists: 두 번째 실행 파일, worlds 설치, -Wall -Wextra -Wpedantic
- 은퇴식: my-turtlesim의 integrate_odom이 물리 엔진에 자리를 물려줌

File: ros2_ws/src/fake_robot/urdf/fake_robot.urdf.xacro (robot description, xacro)
@@ -8,4 +8,46 @@
     <xacro:property name="body_z" value="0.1" />
     <xacro:property name="body_mass" value="5.0" />
+    <gazebo>
+        <plugin filename="gz-sim-joint-state-publisher-system"
+            name="gz::sim::systems::JointStatePublisher">
+        </plugin>
+        <plugin filename="gz-sim-diff-drive-system"
+            name="gz::sim::systems::DiffDrive">
+            <frame_id>odom</frame_id>
+            <child_frame_id>base_link</child_frame_id>
+            <tf_topic>/tf</tf_topic>
+            <left_joint>left_wheel_joint</left_joint>
+            <right_joint>right_wheel_joint</right_joint>
+            <wheel_separation>${track}</wheel_separation>
+            <wheel_radius>${wheel_radius}</wheel_radius>
+            <topic>cmd_vel</topic>
+            <odom_topic>odom</odom_topic>
+            <odom_publish_frequency>30</odom_publish_frequency>
+        </plugin>
+    </gazebo>
+    <gazebo reference="laser">
+        <sensor name="lidar" type="gpu_lidar">
+            <topic>scan</topic>
+            <gz_frame_id>laser</gz_frame_id>
+            <update_rate>10</update_rate>
+            <lidar>
+                <scan>
+                    <horizontal>
+                        <samples>360</samples>
+                        <resolution>1</resolution>
+                        <min_angle>${-pi}</min_angle>
+                        <max_angle>${pi}</max_angle>
+                    </horizontal>
+                </scan>
+                <range>
+                    <min>0.12</min>
+                    <max>10.0</max>
+                    <resolution>0.01</resolution>
+                </range>
+            </lidar>
+            <alwaysOn>1</alwaysOn>
+            <visualize>true</visualize>
+        </sensor>
+    </gazebo>
     <material name="blue">
         <color rgba="0.2 0.4 0.8 1.0" />
@@ -70,4 +112,25 @@
         </joint>
     </xacro:macro>
+    <xacro:macro name="caster" params="prefix x">
+        <link name="${prefix}_caster">
+            <visual>
+                <geometry>
+                    <sphere radius="${caster_radius}" />
+                </geometry>
+                <material name="black" />
+            </visual>
+            <collision>
+                <geometry>
+                    <sphere radius="${caster_radius}" />
+                </geometry>
+            </collision>
+            <xacro:sphere_inertia m="0.1" r="${caster_radius}" />
+        </link>
+        <joint name="${prefix}_caster_joint" type="fixed">
+            <parent link="base_link" />
+            <child link="${prefix}_caster" />
+            <origin xyz="${x} 0 ${-wheel_radius + caster_radius}" rpy="0 0 0" />
+        </joint>
+    </xacro:macro>
     <link name="base_link">
         <visual>
@@ -103,23 +166,6 @@
         <origin xyz="0.2 0 0.1" rpy="0 0 0" />
     </joint>
-    <link name="caster">
-        <visual>
-            <geometry>
-                <sphere radius="${caster_radius}" />
-            </geometry>
-            <material name="black" />
-        </visual>
-        <collision>
-            <geometry>
-                <sphere radius="${caster_radius}" />
-            </geometry>
-        </collision>
-        <xacro:sphere_inertia m="0.1" r="${caster_radius}" />
-    </link>
-    <joint name="caster_joint" type="fixed">
-        <parent link="base_link" />
-        <child link="caster" />
-        <origin xyz="-0.15 0 ${-wheel_radius + caster_radius}" rpy="0 0 0" />
-    </joint>
+    <xacro:caster prefix="front" x="0.15" />
+    <xacro:caster prefix="back" x="-0.15" />
     <xacro:wheel prefix="left" reflect="1" />
     <xacro:wheel prefix="right" reflect="-1" />
